File: Morse Code Emulator.brd (EAGLE design)
At the start: 160.3 x 98.1 mm, 7 parts, among them U1 ARDUINO-UNO-R3-SHIELD

Commit message: commit
Parts:
- added R1: 1k, Tinkercad:RESAD1016W63L850D250B
Connections:
- net U1_D8: now also R1.1
- net U1_GND: now also R1.2
Other:
- board size 160.3 x 98.1 mm -> 160.3 x 118.8 mm
Changed lines of the file:
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@@
 <plain>
 <wire x1="0" y1="0" x2="160.32866319471867" y2="0" width="0" layer="20"/>
-<wire x1="160.32866319471867" y1="0" x2="160.32866319471867" y2="98.14397189914041" width="0" layer="20"/>
-<wire x1="160.32866319471867" y1="98.14397189914041" x2="0" y2="98.14397189914041" width="0" layer="20"/>
-<wire x1="0" y1="98.14397189914041" x2="0" y2="0" width="0" layer="20"/>
+<wire x1="160.32866319471867" y1="0" x2="160.32866319471867" y2="118.79797189914042" width="0" layer="20"/>
+<wire x1="160.32866319471867" y1="118.79797189914042" x2="0" y2="118.79797189914042" width="0" layer="20"/>
+<wire x1="0" y1="118.79797189914042" x2="0" y2="0" width="0" layer="20"/>
 </plain>
 <attributes/>
@@
 </element>
 <element name="R2" library="Tinkercad" package="RESAD1016W63L850D250B" package3d_urn="urn:adsk.eagle:package:31513020/1" value="100" x="36.5172" y="74.268" rot="R90" smashed="yes"/>
+<element name="R1" library="Tinkercad" package="RESAD1016W63L850D250B" package3d_urn="urn:adsk.eagle:package:31513020/1" value="1k" x="51.7572" y="109.828" rot="R90" smashed="yes"/>
 <element name="S1" library="Tinkercad" package="SWITCH-MOMENTARY-PTH-6.5MM" package3d_urn="urn:adsk.eagle:package:32246662/2" value="SWITCH_MOMENTARY" x="49.2172" y="90.778" rot="R90" smashed="yes"/>
 <element name="U1" library="Tinkercad" package="ARDUINO-UNO-R3-SHIELD" package3d_urn="urn:adsk.eagle:package:32092383/3" value="ARDUINO-UNO-R3-SHIELD" x="47.885" y="29.845" rot="R270" smashed="yes"/>
@@
 <contactref element="U1" pad="GND@2"/>
 <contactref element="R3" pad="2"/>
+<contactref element="R1" pad="2"/>
 <wire x1="50.425" y1="5.715" x2="52.965" y2="5.715" width="0" layer="19" extent="1-1"/>
 <wire x1="50.425" y1="5.715" x2="36.455" y2="53.975" width="0" layer="19" extent="1-1"/>
 <wire x1="36.5172" y1="69.188" x2="36.455" y2="53.975" width="0" layer="19" extent="1-1"/>
+<wire x1="36.5172" y1="69.188" x2="51.7572" y2="114.908" width="0" layer="19" extent="1-1"/>
 <wire x1="151.0577" y1="31.4584" x2="52.965" y2="5.715" width="0" layer="19" extent="1-1"/>
 <wire x1="151.0577" y1="31.4584" x2="151.0577" y2="67.0184" width="0" layer="19" extent="1-1"/>
+</signal>
+<signal name="U1_D8">
+<contactref element="S1" pad="3"/>
+<contactref element="U1" pad="D8"/>
+<contactref element="S1" pad="4"/>
+<contactref element="R1" pad="1"/>
+<wire x1="51.4778" y1="87.5268" x2="51.4778" y2="94.0292" width="0" layer="19" extent="1-1"/>
+<wire x1="51.4778" y1="94.0292" x2="51.7572" y2="104.748" width="0" layer="19" extent="1-1"/>
+<wire x1="51.4778" y1="87.5268" x2="51.695" y2="53.975" width="0" layer="19" extent="1-1"/>
 </signal>
 <signal name="U1_5V">
@@
 <wire x1="47.885" y1="5.715" x2="46.9566" y2="87.5268" width="0" layer="19" extent="1-1"/>
 </signal>
-<signal name="U1_D8">
-<contactref element="S1" pad="3"/>
-<contactref element="U1" pad="D8"/>
-<contactref element="S1" pad="4"/>
-<wire x1="51.4778" y1="87.5268" x2="51.4778" y2="94.0292" width="0" layer="19" extent="1-1"/>
-<wire x1="51.4778" y1="87.5268" x2="51.695" y2="53.975" width="0" layer="19" extent="1-1"/>
-</signal>
 <signal name="U1_D12">
